File: circuit/scem/scem.kicad_sch (KiCad schematic)
At the start: 1 part, among them U1 ATmega328P-P U

Commit message: test
Parts:
- removed U1: ATmega328P-P U, Package_DIP:DIP-28_W7.62mm, symbol MCU_Microchip_ATmega:ATmega328P-P
Changed lines of the file:
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@@
     (title "afanci")
-  )
-  (symbol (lib_id "MCU_Microchip_ATmega:ATmega328P-P") (at 43.18 54.61 0) (unit 1)
-    (in_bom yes) (on_board yes) (dnp no)
-    (property "Reference" "U1" (at 21.59 20.4821 0)
-      (effects (font (size 1.27 1.27)))
-    )
-    (property "Value" "ATmega328P-P U" (at 29.21 15.24 0)
-      (effects (font (size 1.27 1.27)))
-    )
-    (property "Footprint" "Package_DIP:DIP-28_W7.62mm" (at 43.18 54.61 0)
-      (effects (font (size 1.27 1.27) italic) hide)
-    )
-    (property "Datasheet" "http://ww1.microchip.com/downloads/en/DeviceDoc/ATmega328_P%20AVR%20MCU%20with%20picoPower%20Technology%20Data%20Sheet%2040001984A.pdf" (at 43.18 54.61 0)
-      (effects (font (size 1.27 1.27)) hide)
-    )
-    (pin "1")
-    (pin "10")
-    (pin "11")
-    (pin "12")
-    (pin "13")
-    (pin "14")
-    (pin "15")
-    (pin "16")
-    (pin "17")
-    (pin "18")
-    (pin "19")
-    (pin "2")
-    (pin "20")
-    (pin "21")
-    (pin "22")
-    (pin "23")
-    (pin "24")
-    (pin "25")
-    (pin "26")
-    (pin "27")
-    (pin "28")
-    (pin "3")
-    (pin "4")
-    (pin "5")
-    (pin "6")
-    (pin "7")
-    (pin "8")
-    (pin "9")
-    (instances
-      (project "scem"
-        (path "/60d66d5a-e0e3-4631-84c8-aa9e13baae05"
-          (reference "U1") (unit 1)
-        )
-      )
-    )
   )
   (sheet_instances

Commit message: man ey
Parts:
- added 16mhz: Crystal, symbol Device:Crystal
- added U1: ATmega328-P, Package_DIP:DIP-28_W7.62mm, symbol MCU_Microchip_ATmega:ATmega328-P
Connections:
- new net +5V: U1.7 (VCC)
- new net GND: U1.22 (GND), U1.8 (GND)
Changed lines of the file:
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@@
     (title "afanci")
+  )
+  (wire (pts (xy 17.78 19.05) (xy 17.78 30.48))
+    (stroke (width 0) (type default))
+  )
+  (wire (pts (xy 44.45 115.57) (xy 44.45 106.68))
+    (stroke (width 0) (type default))
+  )
+  (wire (pts (xy 17.78 30.48) (xy 44.45 30.48))
+    (stroke (width 0) (type default))
+  )
+  (wire (pts (xy 19.05 115.57) (xy 44.45 115.57))
+    (stroke (width 0) (type default))
+  )
+  (symbol (lib_id "power:+5V") (at 17.78 19.05 0) (unit 1)
+    (in_bom yes) (on_board yes) (dnp no) (fields_autoplaced)
+    (property "Reference" "#PWR01" (at 17.78 22.86 0)
+      (effects (font (size 1.27 1.27)) hide)
+    )
+    (property "Value" "+5V" (at 17.78 13.97 0)
+      (effects (font (size 1.27 1.27)))
+    )
+    (property "Footprint" "" (at 17.78 19.05 0)
+      (effects (font (size 1.27 1.27)) hide)
+    )
+    (property "Datasheet" "" (at 17.78 19.05 0)
+      (effects (font (size 1.27 1.27)) hide)
+    )
+    (pin "1")
+    (instances
+      (project "scem"
+        (path "/60d66d5a-e0e3-4631-84c8-aa9e13baae05"
+          (reference "#PWR01") (unit 1)
+        )
+      )
+    )
+  )
+  (symbol (lib_id "MCU_Microchip_ATmega:ATmega328-P") (at 44.45 68.58 0) (unit 1)
+    (in_bom yes) (on_board yes) (dnp no) (fields_autoplaced)
+    (property "Reference" "U1" (at 22.86 34.4521 0)
+      (effects (font (size 1.27 1.27)))
+    )
+    (property "Value" "ATmega328-P" (at 22.86 36.9921 0)
+      (effects (font (size 1.27 1.27)))
+    )
+    (property "Footprint" "Package_DIP:DIP-28_W7.62mm" (at 44.45 68.58 0)
+      (effects (font (size 1.27 1.27) italic) hide)
+    )
+    (property "Datasheet" "http://ww1.microchip.com/downloads/en/DeviceDoc/ATmega328_P%20AVR%20MCU%20with%20picoPower%20Technology%20Data%20Sheet%2040001984A.pdf" (at 44.45 68.58 0)
+      (effects (font (size 1.27 1.27)) hide)
+    )
+    (pin "1")
+    (pin "10")
+    (pin "11")
+    (pin "12")
+    (pin "13")
+    (pin "14")
+    (pin "15")
+    (pin "16")
+    (pin "17")
+    (pin "18")
+    (pin "19")
+    (pin "2")
+    (pin "20")
+    (pin "21")
+    (pin "22")
+    (pin "23")
+    (pin "24")
+    (pin "25")
+    (pin "26")
+    (pin "27")
+    (pin "28")
+    (pin "3")
+    (pin "4")
+    (pin "5")
+    (pin "6")
+    (pin "7")
+    (pin "8")
+    (pin "9")
+    (instances
+      (project "scem"
+        (path "/60d66d5a-e0e3-4631-84c8-aa9e13baae05"
+          (reference "U1") (unit 1)
+        )
+      )
+    )
+  )
+  (symbol (lib_id "Device:Crystal") (at 68.58 25.4 0) (unit 1)
+    (in_bom yes) (on_board yes) (dnp no) (fields_autoplaced)
+    (property "Reference" "16mhz" (at 68.58 17.78 0)
+      (effects (font (size 1.27 1.27)))
+    )
+    (property "Value" "Crystal" (at 68.58 20.32 0)
+      (effects (font (size 1.27 1.27)))
+    )
+    (property "Footprint" "" (at 68.58 25.4 0)
+      (effects (font (size 1.27 1.27)) hide)
+    )
+    (property "Datasheet" "~" (at 68.58 25.4 0)
+      (effects (font (size 1.27 1.27)) hide)
+    )
+    (pin "1")
+    (pin "2")
+    (instances
+      (project "scem"
+        (path "/60d66d5a-e0e3-4631-84c8-aa9e13baae05"
+          (reference "16mhz") (unit 1)
+        )
+      )
+    )
+  )
+  (symbol (lib_id "power:+12V") (at 24.13 19.05 0) (unit 1)
+    (in_bom yes) (on_board yes) (dnp no) (fields_autoplaced)
+    (property "Reference" "#PWR02" (at 24.13 22.86 0)
+      (effects (font (size 1.27 1.27)) hide)
+    )
+    (property "Value" "+12V" (at 24.13 13.97 0)
+      (effects (font (size 1.27 1.27)))
+    )
+    (property "Footprint" "" (at 24.13 19.05 0)
+      (effects (font (size 1.27 1.27)) hide)
+    )
+    (property "Datasheet" "" (at 24.13 19.05 0)
+      (effects (font (size 1.27 1.27)) hide)
+    )
+    (pin "1")
+    (instances
+      (project "scem"
+        (path "/60d66d5a-e0e3-4631-84c8-aa9e13baae05"
+          (reference "#PWR02") (unit 1)
+        )
+      )
+    )
+  )
+  (symbol (lib_id "power:GND") (at 19.05 115.57 0) (unit 1)
+    (in_bom yes) (on_board yes) (dnp no) (fields_autoplaced)
+    (property "Reference" "#PWR03" (at 19.05 121.92 0)
+      (effects (font (size 1.27 1.27)) hide)
+    )
+    (property "Value" "GND" (at 19.05 120.65 0)
+      (effects (font (size 1.27 1.27)))
+    )
+    (property "Footprint" "" (at 19.05 115.57 0)
+      (effects (font (size 1.27 1.27)) hide)
+    )
+    (property "Datasheet" "" (at 19.05 115.57 0)
+      (effects (font (size 1.27 1.27)) hide)
+    )
+    (pin "1")
+    (instances
+      (project "scem"
+        (path "/60d66d5a-e0e3-4631-84c8-aa9e13baae05"
+          (reference "#PWR03") (unit 1)
+        )
+      )
+    )
   )
   (sheet_instances

Commit message: test
Parts:
- removed 16mhz: Crystal, symbol Device:Crystal
- removed U1: ATmega328-P, Package_DIP:DIP-28_W7.62mm, symbol MCU_Microchip_ATmega:ATmega328-P
Changed lines of the file:
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@@
     (title "afanci")
-  )
-  (wire (pts (xy 17.78 19.05) (xy 17.78 30.48))
-    (stroke (width 0) (type default))
-  )
-  (wire (pts (xy 44.45 115.57) (xy 44.45 106.68))
-    (stroke (width 0) (type default))
-  )
-  (wire (pts (xy 17.78 30.48) (xy 44.45 30.48))
-    (stroke (width 0) (type default))
-  )
-  (wire (pts (xy 19.05 115.57) (xy 44.45 115.57))
-    (stroke (width 0) (type default))
-  )
-  (symbol (lib_id "power:+5V") (at 17.78 19.05 0) (unit 1)
-    (in_bom yes) (on_board yes) (dnp no) (fields_autoplaced)
-    (property "Reference" "#PWR01" (at 17.78 22.86 0)
-      (effects (font (size 1.27 1.27)) hide)
-    )
-    (property "Value" "+5V" (at 17.78 13.97 0)
-      (effects (font (size 1.27 1.27)))
-    )
-    (property "Footprint" "" (at 17.78 19.05 0)
-      (effects (font (size 1.27 1.27)) hide)
-    )
-    (property "Datasheet" "" (at 17.78 19.05 0)
-      (effects (font (size 1.27 1.27)) hide)
-    )
-    (pin "1")
-    (instances
-      (project "scem"
-        (path "/60d66d5a-e0e3-4631-84c8-aa9e13baae05"
-          (reference "#PWR01") (unit 1)
-        )
-      )
-    )
-  )
-  (symbol (lib_id "MCU_Microchip_ATmega:ATmega328-P") (at 44.45 68.58 0) (unit 1)
-    (in_bom yes) (on_board yes) (dnp no) (fields_autoplaced)
-    (property "Reference" "U1" (at 22.86 34.4521 0)
-      (effects (font (size 1.27 1.27)))
-    )
-    (property "Value" "ATmega328-P" (at 22.86 36.9921 0)
-      (effects (font (size 1.27 1.27)))
-    )
-    (property "Footprint" "Package_DIP:DIP-28_W7.62mm" (at 44.45 68.58 0)
-      (effects (font (size 1.27 1.27) italic) hide)
-    )
-    (property "Datasheet" "http://ww1.microchip.com/downloads/en/DeviceDoc/ATmega328_P%20AVR%20MCU%20with%20picoPower%20Technology%20Data%20Sheet%2040001984A.pdf" (at 44.45 68.58 0)
-      (effects (font (size 1.27 1.27)) hide)
-    )
-    (pin "1")
-    (pin "10")
-    (pin "11")
-    (pin "12")
-    (pin "13")
-    (pin "14")
-    (pin "15")
-    (pin "16")
-    (pin "17")
-    (pin "18")
-    (pin "19")
-    (pin "2")
-    (pin "20")
-    (pin "21")
-    (pin "22")
-    (pin "23")
-    (pin "24")
-    (pin "25")
-    (pin "26")
-    (pin "27")
-    (pin "28")
-    (pin "3")
-    (pin "4")
-    (pin "5")
-    (pin "6")
-    (pin "7")
-    (pin "8")
-    (pin "9")
-    (instances
-      (project "scem"
-        (path "/60d66d5a-e0e3-4631-84c8-aa9e13baae05"
-          (reference "U1") (unit 1)
-        )
-      )
-    )
-  )
-  (symbol (lib_id "Device:Crystal") (at 68.58 25.4 0) (unit 1)
-    (in_bom yes) (on_board yes) (dnp no) (fields_autoplaced)
-    (property "Reference" "16mhz" (at 68.58 17.78 0)
-      (effects (font (size 1.27 1.27)))
-    )
-    (property "Value" "Crystal" (at 68.58 20.32 0)
-      (effects (font (size 1.27 1.27)))
-    )
-    (property "Footprint" "" (at 68.58 25.4 0)
-      (effects (font (size 1.27 1.27)) hide)
-    )
-    (property "Datasheet" "~" (at 68.58 25.4 0)
-      (effects (font (size 1.27 1.27)) hide)
-    )
-    (pin "1")
-    (pin "2")
-    (instances
-      (project "scem"
-        (path "/60d66d5a-e0e3-4631-84c8-aa9e13baae05"
-          (reference "16mhz") (unit 1)
-        )
-      )
-    )
-  )
-  (symbol (lib_id "power:+12V") (at 24.13 19.05 0) (unit 1)
-    (in_bom yes) (on_board yes) (dnp no) (fields_autoplaced)
-    (property "Reference" "#PWR02" (at 24.13 22.86 0)
-      (effects (font (size 1.27 1.27)) hide)
-    )
-    (property "Value" "+12V" (at 24.13 13.97 0)
-      (effects (font (size 1.27 1.27)))
-    )
-    (property "Footprint" "" (at 24.13 19.05 0)
-      (effects (font (size 1.27 1.27)) hide)
-    )
-    (property "Datasheet" "" (at 24.13 19.05 0)
-      (effects (font (size 1.27 1.27)) hide)
-    )
-    (pin "1")
-    (instances
-      (project "scem"
-        (path "/60d66d5a-e0e3-4631-84c8-aa9e13baae05"
-          (reference "#PWR02") (unit 1)
-        )
-      )
-    )
-  )
-  (symbol (lib_id "power:GND") (at 19.05 115.57 0) (unit 1)
-    (in_bom yes) (on_board yes) (dnp no) (fields_autoplaced)
-    (property "Reference" "#PWR03" (at 19.05 121.92 0)
-      (effects (font (size 1.27 1.27)) hide)
-    )
-    (property "Value" "GND" (at 19.05 120.65 0)
-      (effects (font (size 1.27 1.27)))
-    )
-    (property "Footprint" "" (at 19.05 115.57 0)
-      (effects (font (size 1.27 1.27)) hide)
-    )
-    (property "Datasheet" "" (at 19.05 115.57 0)
-      (effects (font (size 1.27 1.27)) hide)
-    )
-    (pin "1")
-    (instances
-      (project "scem"
-        (path "/60d66d5a-e0e3-4631-84c8-aa9e13baae05"
-          (reference "#PWR03") (unit 1)
-        )
-      )
-    )
   )
   (sheet_instances
